File: Hardware/VersaTerm.kicad_sch (KiCad schematic)
At the start: 60 parts, among them J101 USB_C_Receptacle_PowerOnly_6P, J102 Serial, J103 VTTL, J104 Mini-DIN-6, J105 DE15_Receptacle_HighDensity, J106 USB Keyboard, J107 RS232, J108 HDMI_A, Q101 BSS138, Q102 BSS138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

Commit message: finalized PCB
Parts:
- removed J101: USB_C_Receptacle_PowerOnly_6P, Connector_USB:USB_C_Receptacle_GCT_USB4125-xx-x-0190_6P_TopMnt_Horizontal, symbol Connector:USB_C_Receptacle_PowerOnly_6P
- added J101: USB_C_Receptacle_USB2.0_16P, Connector_USB:USB_C_Receptacle_G-Switch_GT-USB-7010ASV, symbol Connector:USB_C_Receptacle_USB2.0_16P
- added J102: USB Keyboard, Connector_USB:USB_A_CONNFLY_DS1095-WNR0, symbol Connector:USB_A
- added R131, R132: 1k, Resistor_SMD:R_0805_2012Metric, symbol Device:R
- SW101, SW102: footprint Button_Switch_SMD:SW_SPST_TL3342 -> Button_Switch_THT:SW_SPST_Omron_B3F-315x_Angled
- renumbered J102 to J104, J104 to J105, J105 to J106, J106 to J107, J107 to J108, J108 to J109
Connections:
- net +5V: now also J101.A4 (VBUS), J101.A9 (VBUS), J101.B4 (VBUS), J101.B9 (VBUS), J102.1 (VBUS)
- net GND: now also J101.A1 (GND), J101.A12 (GND), J101.B1 (GND), J101.B12 (GND), J101.S1 (SHIELD), J102.4 (GND), J102.5 (Shield)
- net RTS: now also R132.1; no longer Q105.1 (G)
- net TX: now also R131.1; no longer Q104.1 (G)
- net _D0-: now reaches J109.9 (D0-), R126.1
- net _D1+: now reaches J109.4 (D1+), R123.1
- net _D1-: now reaches J109.6 (D1-), R124.1
- net _D2+: now reaches J109.1 (D2+), R121.1
- net _CK+: now reaches J109.10 (CK+), R127.1
- net _CK-: now reaches J109.12 (CK-), R128.1
- net _D2-: now reaches J109.3 (D2-), R122.1
- net _D0+: now reaches J109.7 (D0+), R125.1
- net K+: now reaches J107.3 (D+)
- net K+: now also U102.3 (I/O2); no longer U102.1 (I/O1)
- net K-: now reaches J107.2 (D-)
- net K-: now also U102.1 (I/O1); no longer U102.3 (I/O2)
- net Pi Pico/USB+ renamed K1-
- net Pi Pico/USB- renamed K1+
- new net: Q105.1 (G), R132.2
- new net: Q104.1 (G), R131.2
- no-connect marks 19 -> 27
Other:
- moved on the sheet: J103, R121, R122, R123, R124, R125, R126, R127, R128

Commit message: updated version not final reviewed
Parts:
- added R1: 2k2, Resistor_SMD:R_0805_2012Metric, symbol Device:R
- added R2, R3: 5k1, Resistor_SMD:R_0805_2012Metric, symbol Device:R
Connections:
- net GND: now also R1.1, R2.2, R3.2
- net at Q101.1 (G), R103.2: now also R1.2
- net at J101.A5 (CC1): now also R2.1
- net at J101.B5 (CC2): now also R3.1
- no-connect marks 27 -> 25
Other:
- moved on the sheet: R103, R121, R122, R123, R124, R125, R126, R127, R128

Commit message: rework
Parts:
- removed J107: USB Keyboard, Connector_USB:USB_A_CONNFLY_DS1095-WNR0, symbol Connector:USB_A
- removed U102: USBLC6-2SC6, Package_TO_SOT_SMD:SOT-23-6, symbol Power_Protection:USBLC6-2SC6
- J102: value USB Keyboard -> Power
Other:
- sheet Pi Pico ports: added none; removed USB+, USB-
