File: Hardware/pico.kicad_sch (KiCad schematic)
At the start: 38 parts, among them J201 USB_C_Receptacle_USB2.0_16P, J202 Conn_01x03, Q201 DMG1012T, SW201 SW_SPST, U201 USBLC6-2SC6, U202 W25Q16JVSS, U203 RP2040, Y201 12MHz

Commit message: finalized PCB
Parts:
- Q201: footprint Package_TO_SOT_SMD:SOT-523 -> Package_TO_SOT_SMD:SOT-323_SC-70
- SW201: footprint Buzzer_Beeper:Buzzer_Mallory_AST1240MLQ -> Button_Switch_THT:SW_SPST_Omron_B3F-315x_Angled
- U203: footprint Package_DFN_QFN:QFN-56-1EP_7x7mm_P0.4mm_EP3.2x3.2mm -> Package_DFN_QFN:QFN-56-1EP_7x7mm_P0.4mm_EP3.2x3.2mm_ThermalVias
Changed lines of the file:
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@@
 			)
 		)
-		(property "Footprint" "Package_DFN_QFN:QFN-56-1EP_7x7mm_P0.4mm_EP3.2x3.2mm"
+		(property "Footprint" "Package_DFN_QFN:QFN-56-1EP_7x7mm_P0.4mm_EP3.2x3.2mm_ThermalVias"
 			(at 111.76 130.81 0)
 			(effects
@@
 			)
 		)
-		(property "Footprint" "Package_TO_SOT_SMD:SOT-523"
+		(property "Footprint" "Package_TO_SOT_SMD:SOT-323_SC-70"
 			(at 156.845 171.45 0)
 			(effects
@@
 			)
 		)
-		(property "Footprint" "Buzzer_Beeper:Buzzer_Mallory_AST1240MLQ"
+		(property "Footprint" "Button_Switch_THT:SW_SPST_Omron_B3F-315x_Angled"
 			(at 45.72 92.71 0)
 			(effects

Commit message: updated version not final reviewed
Changed lines of the file:
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@@
 	(wire
 		(pts
-			(xy 48.26 21.59) (xy 48.26 22.86)
+			(xy 58.42 21.59) (xy 58.42 22.86)
 		)
 		(stroke
@@
 	(wire
 		(pts
+			(xy 44.45 22.86) (xy 58.42 22.86)
+		)
+		(stroke
+			(width 0)
+			(type default)
+		)
+	)
+	(wire
+		(pts
 			(xy 80.01 31.75) (xy 80.01 33.02)
 		)
@@
 	(wire
 		(pts
-			(xy 48.26 22.86) (xy 44.45 22.86)
-		)
-		(stroke
-			(width 0)
-			(type default)
-		)
-	)
-	(wire
-		(pts
 			(xy 63.5 100.33) (xy 66.04 100.33)
 		)
@@
 		(on_board yes)
 		(dnp no)
-		(fields_autoplaced yes)
 		(property "Reference" "#PWR0234"
 			(at 25.4 172.72 0)
@@
 		)
 		(property "Value" "+3V3"
-			(at 25.4 163.83 0)
+			(at 25.4 165.1 0)
 			(effects
 				(font
@@
 		(dnp no)
 		(property "Reference" "R211"
-			(at 83.058 147.574 90)
+			(at 78.74 146.05 90)
 			(effects
 				(font
@@
 		(on_board yes)
 		(dnp no)
-		(fields_autoplaced yes)
 		(property "Reference" "#PWR0247"
 			(at 55.88 185.42 0)
@@
 		)
 		(property "Value" "GND"
-			(at 55.88 184.15 0)
+			(at 55.88 182.88 0)
 			(effects
 				(font
@@
 		(on_board yes)
 		(dnp no)
-		(fields_autoplaced yes)
 		(property "Reference" "#PWR0230"
 			(at 30.48 162.56 0)
@@
 		)
 		(property "Value" "GND"
-			(at 30.48 161.29 0)
+			(at 30.48 160.02 0)
 			(effects
 				(font
@@
 		(on_board yes)
 		(dnp no)
-		(fields_autoplaced yes)
 		(property "Reference" "#PWR0244"
 			(at 33.02 185.42 0)
@@
 		)
 		(property "Value" "GND"
-			(at 33.02 184.15 0)
+			(at 33.02 182.88 0)
 			(effects
 				(font
@@
 		(on_board yes)
 		(dnp no)
-		(fields_autoplaced yes)
 		(property "Reference" "#PWR0223"
 			(at 17.78 149.86 0)
@@
 		)
 		(property "Value" "+3V3"
-			(at 17.78 140.97 0)
+			(at 17.78 142.24 0)
 			(effects
 				(font
@@
 		(on_board yes)
 		(dnp no)
-		(fields_autoplaced yes)
 		(property "Reference" "#PWR0220"
 			(at 24.13 107.95 0)
@@
 		)
 		(property "Value" "+3V3"
-			(at 24.13 99.06 0)
+			(at 24.13 100.33 0)
 			(effects
 				(font
@@
 		(on_board yes)
 		(dnp no)
-		(fields_autoplaced yes)
 		(property "Reference" "#PWR0235"
 			(at 33.02 172.72 0)
@@
 		)
 		(property "Value" "+3V3"
-			(at 33.02 163.83 0)
+			(at 33.02 165.1 0)
 			(effects
 				(font
@@
 		(on_board yes)
 		(dnp no)
-		(fields_autoplaced yes)
 		(property "Reference" "#PWR0243"
 			(at 25.4 185.42 0)
@@
 		)
 		(property "Value" "GND"
-			(at 25.4 184.15 0)
+			(at 25.4 182.88 0)
 			(effects
 				(font
@@
 		(on_board yes)
 		(dnp no)
-		(fields_autoplaced yes)
 		(property "Reference" "#PWR0239"
 			(at 63.5 172.72 0)
@@
 		)
 		(property "Value" "+3V3"
-			(at 63.5 163.83 0)
+			(at 63.5 165.1 0)
 			(effects
 				(font
@@
 		(dnp no)
 		(property "Reference" "R209"
-			(at 37.084 98.552 90)
+			(at 36.83 97.155 90)
 			(effects
 				(font
@@
 		(on_board yes)
 		(dnp no)
-		(fields_autoplaced yes)
 		(property "Reference" "#PWR0237"
 			(at 48.26 172.72 0)
@@
 		)
 		(property "Value" "+3V3"
-			(at 48.26 163.83 0)
+			(at 48.26 165.1 0)
 			(effects
 				(font
@@
 		(on_board yes)
 		(dnp no)
-		(fields_autoplaced yes)
 		(property "Reference" "#PWR0238"
 			(at 55.88 172.72 0)
@@
 		)
 		(property "Value" "+3V3"
-			(at 55.88 163.83 0)
+			(at 55.88 165.1 0)
 			(effects
 				(font
@@
 		(on_board yes)
 		(dnp no)
-		(fields_autoplaced yes)
 		(property "Reference" "#PWR0236"
 			(at 40.64 172.72 0)
@@
 		)
 		(property "Value" "+3V3"
-			(at 40.64 163.83 0)
+			(at 40.64 165.1 0)
 			(effects
 				(font
@@
 		(on_board yes)
 		(dnp no)
-		(fields_autoplaced yes)
 		(property "Reference" "#PWR0224"
 			(at 30.48 149.86 0)
@@
 		)
 		(property "Value" "+3V3"
-			(at 30.48 140.97 0)
+			(at 30.48 142.24 0)
 			(effects
 				(font
@@
 		(on_board yes)
 		(dnp no)
-		(fields_autoplaced yes)
 		(property "Reference" "#PWR0221"
 			(at 24.13 138.43 0)
@@
 		)
 		(property "Value" "GND"
-			(at 24.13 137.16 0)
+			(at 24.13 135.89 0)
 			(effects
 				(font
@@
 		(on_board yes)
 		(dnp no)
-		(fields_autoplaced yes)
 		(property "Reference" "#PWR0248"
 			(at 63.5 185.42 0)
@@
 		)
 		(property "Value" "GND"
-			(at 63.5 184.15 0)
+			(at 63.5 182.88 0)
 			(effects
 				(font
@@
 	(symbol
 		(lib_id "power:+5V")
-		(at 48.26 21.59 0)
+		(at 58.42 21.59 0)
 		(unit 1)
 		(exclude_from_sim no)
@@
 		(fields_autoplaced yes)
 		(property "Reference" "#PWR0201"
-			(at 48.26 25.4 0)
+			(at 58.42 25.4 0)
 			(effects
 				(font
@@
 		)
 		(property "Value" "+5V"
-			(at 48.26 16.51 0)
+			(at 58.42 16.51 0)
 			(effects
 				(font
@@
 		)
 		(property "Footprint" ""
-			(at 48.26 21.59 0)
+			(at 58.42 21.59 0)
 			(effects
 				(font
@@
 		)
 		(property "Datasheet" ""
-			(at 48.26 21.59 0)
+			(at 58.42 21.59 0)
 			(effects
 				(font
@@
 		)
 		(property "Description" "Power symbol creates a global label with name \"+5V\""
-			(at 48.26 21.59 0)
+			(at 58.42 21.59 0)
 			(effects
 				(font
@@
 		(on_board yes)
 		(dnp no)
-		(fields_autoplaced yes)
 		(property "Reference" "#PWR0242"
 			(at 17.78 185.42 0)
@@
 		)
 		(property "Value" "GND"
-			(at 17.78 184.15 0)
+			(at 17.78 182.88 0)
 			(effects
 				(font
@@
 		(on_board yes)
 		(dnp no)
-		(fields_autoplaced yes)
 		(property "Reference" "#PWR0245"
 			(at 40.64 185.42 0)
@@
 		)
 		(property "Value" "GND"
-			(at 40.64 184.15 0)
+			(at 40.64 182.88 0)
 			(effects
 				(font
@@
 		(on_board yes)
 		(dnp no)
-		(fields_autoplaced yes)
 		(property "Reference" "#PWR0246"
 			(at 48.26 185.42 0)
@@
 		)
 		(property "Value" "GND"
-			(at 48.26 184.15 0)
+			(at 48.26 182.88 0)
 			(effects
 				(font
@@
 		(on_board yes)
 		(dnp no)
-		(fields_autoplaced yes)
 		(property "Reference" "#PWR0229"
 			(at 17.78 162.56 0)
@@
 		)
 		(property "Value" "GND"
-			(at 17.78 161.29 0)
+			(at 17.78 160.02 0)
 			(effects
 				(font
@@
 		(on_board yes)
 		(dnp no)
-		(fields_autoplaced yes)
 		(property "Reference" "#PWR0233"
 			(at 17.78 172.72 0)
@@
 		)
 		(property "Value" "+3V3"
-			(at 17.78 163.83 0)
+			(at 17.78 165.1 0)
 			(effects
 				(font

Commit message: rework
Parts:
- Y201: footprint Crystal:Crystal_SMD_Abracon_ABM3B-4Pin_5.0x3.2mm -> Crystal:Crystal_SMD_3225-4Pin_3.2x2.5mm
Changed lines of the file:
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@@
 	)
 	(junction
-		(at 63.5 100.33)
-		(diameter 0)
-		(color 0 0 0 0)
-	)
-	(junction
 		(at 68.58 148.59)
 		(diameter 0)
@@
 	)
 	(junction
-		(at 63.5 102.87)
-		(diameter 0)
-		(color 0 0 0 0)
-	)
-	(junction
 		(at 116.84 81.28)
 		(diameter 0)
@@
 	(wire
 		(pts
-			(xy 63.5 102.87) (xy 66.04 102.87)
+			(xy 60.96 102.87) (xy 66.04 102.87)
 		)
 		(stroke
@@
 	(wire
 		(pts
-			(xy 62.23 106.68) (xy 63.5 106.68)
-		)
-		(stroke
-			(width 0)
-			(type default)
-		)
-	)
-	(wire
-		(pts
 			(xy 148.59 102.87) (xy 137.16 102.87)
 		)
@@
 	(wire
 		(pts
-			(xy 60.96 100.33) (xy 63.5 100.33)
+			(xy 60.96 100.33) (xy 66.04 100.33)
 		)
 		(stroke
@@
 	(wire
 		(pts
-			(xy 63.5 106.68) (xy 63.5 102.87)
-		)
-		(stroke
-			(width 0)
-			(type default)
-		)
-	)
-	(wire
-		(pts
 			(xy 73.66 102.87) (xy 86.36 102.87)
 		)
@@
 	(wire
 		(pts
-			(xy 60.96 102.87) (xy 63.5 102.87)
-		)
-		(stroke
-			(width 0)
-			(type default)
-		)
-	)
-	(wire
-		(pts
 			(xy 242.57 24.13) (xy 242.57 26.67)
 		)
@@
 	(wire
 		(pts
-			(xy 63.5 100.33) (xy 66.04 100.33)
-		)
-		(stroke
-			(width 0)
-			(type default)
-		)
-	)
-	(wire
-		(pts
 			(xy 38.1 99.06) (xy 38.1 92.71)
 		)
@@
 	(wire
 		(pts
-			(xy 63.5 96.52) (xy 63.5 100.33)
-		)
-		(stroke
-			(width 0)
-			(type default)
-		)
-	)
-	(wire
-		(pts
 			(xy 49.53 138.43) (xy 48.26 138.43)
 		)
@@
 	(wire
 		(pts
-			(xy 62.23 96.52) (xy 63.5 96.52)
-		)
-		(stroke
-			(width 0)
-			(type default)
-		)
-	)
-	(wire
-		(pts
 			(xy 148.59 166.37) (xy 137.16 166.37)
 		)
@@
 		)
 	)
-	(hierarchical_label "USB+"
-		(shape input)
-		(at 62.23 106.68 180)
-		(fields_autoplaced yes)
-		(effects
-			(font
-				(size 1.27 1.27)
-			)
-			(justify right)
-		)
-	)
 	(hierarchical_label "GPIO3"
 		(shape input)
@@
 		)
 	)
-	(hierarchical_label "USB-"
-		(shape input)
-		(at 62.23 96.52 180)
-		(fields_autoplaced yes)
-		(effects
-			(font
-				(size 1.27 1.27)
-			)
-			(justify right)
-		)
-	)
 	(hierarchical_label "GPIO6"
 		(shape input)
@@
 			)
 		)
-		(property "Footprint" "Crystal:Crystal_SMD_Abracon_ABM3B-4Pin_5.0x3.2mm"
+		(property "Footprint" "Crystal:Crystal_SMD_3225-4Pin_3.2x2.5mm"
 			(at 68.58 143.51 0)
 			(effects
