File: Hardware/VersaTerm.kicad_pcb (KiCad board)
At the start: 4 copper layers, 165 x 125 mm, 122 parts, among them J101 USB_C_Receptacle_USB2.0_16P, J102 USB Keyboard, J103 VTTL, J104 Serial, J105 Mini-DIN-6, J106 DE15_Receptacle_HighDensity, J107 USB Keyboard, J108 RS232, J109 HDMI_A, J201 USB_C_Receptacle_USB2.0_16P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

Commit message: pcb update
Routing:
- net /Pi Pico/RUN: track 95.8 -> 95.2 mm
- net +5V: vias 251 -> 252
Other:
- board text added: "VersaTerm"
- board text removed: "VersTerm"

Commit message: updated version not final reviewed
Parts:
- added R1: 2k2, Resistor_SMD:R_0805_2012Metric, F.Cu at (188.2, 121.9)
- added R2: 5k1, Resistor_SMD:R_0805_2012Metric, F.Cu at (129.8, 42.4)
- added R3: 5k1, Resistor_SMD:R_0805_2012Metric, F.Cu at (126.8, 42.4)
- added U2: FSUSB42MUX, Package_SO:MSOP-10_3x3mm_P0.5mm, F.Cu at (141.5, 112.1)
- moved C303 6.89 mm to (131.6, 49.3), turned to 90 degrees
- moved C302 5.73 mm to (129.5, 49.3), turned to 90 degrees
Connections:
- J101 pad A5: unconnected-(J101-CC1-PadA5) -> Net-(J101-CC1)
- J101 pad B5: unconnected-(J101-CC2-PadB5) -> Net-(J101-CC2)
Routing:
- net +3V3: track 230.3 -> 241.2 mm
- net /CK-: track 75.6 -> 83.5 mm
- net /CK+: track 77.8 -> 85.8 mm
- net Net-(J101-CC1): track 0.00 -> 3.47 mm
- net Net-(J101-CC2): track 0.00 -> 3.45 mm
- net GND: track 107.7 -> 110.7 mm, vias 73 -> 76
- net Net-(Q101-G): track 2.00 -> 3.84 mm
- net Net-(U301-FB): track 17.5 -> 18.5 mm
- net /D1-: track 88.1 -> 87.5 mm
- net +5V: vias 252 -> 250

Commit message: rework
Parts:
- removed J107: USB Keyboard, Connector_USB:USB_A_CONNFLY_DS1095-WNR0
- removed U102: USBLC6-2SC6, Package_TO_SOT_SMD:SOT-23-6
- removed U2: FSUSB42MUX, Package_SO:MSOP-10_3x3mm_P0.5mm
- J102: value USB Keyboard -> Power
- Y201: footprint Crystal:Crystal_SMD_Abracon_ABM3B-4Pin_5.0x3.2mm -> Crystal:Crystal_SMD_3225-4Pin_3.2x2.5mm
- moved C204 4.05 mm to (150.1, 77.3), turned to 90 degrees
- moved C205 3.78 mm to (147.8, 77.3)
- moved Y201 1.49 mm to (149.0, 80.8), turned to 0 degrees
Routing:
- net /K1+: track 179.2 -> 98.1 mm
- net /K1-: track 180.0 -> 99.7 mm
- net /K-: track 7.22 -> 0.00 mm
- net /K+: track 7.22 -> 0.00 mm
- net GND: track 110.7 -> 103.7 mm
- net Net-(C205-Pad1): track 10.1 -> 6.30 mm
- net +5V: track 26.6 -> 25.5 mm, vias 250 -> 235
- net Net-(U203-XIN): track 9.17 -> 10.1 mm
Other:
- board text added: "USB Connection"
- board text removed: "KEYBOARD"
- board text removed: "Terminal"

Commit message: Final Review Version (Update USB Routing)
Parts:
- added G***: LOGO, TheBrutzlers_Lib:approved_theBrutzler, F.Cu at (150.4, 117.8)
- added G***: LOGO, TheBrutzlers_Lib:thebrutzler_approved_small02, F.Cu at (95.0, 41.8)
Routing:
- net /Pi Pico/USB_P: track 12.3 -> 8.28 mm, vias 2 -> 0
- net /Pi Pico/USB_N: track 11.9 -> 9.06 mm, vias 2 -> 0
- net GND: vias 76 -> 75
